File: hardware/THT-PCB/usb3sun-THT.kicad_pcb (KiCad board)
At the start: 2 copper layers, 0 parts

Commit message: SCH Complete; Begin PCB work!
Parts:
- added BZ1: SEA-1285F, Buzzer_Beeper:Buzzer_12x9.5RM7.6, F.Cu at (75.5, 102.3)
- added C1: 100uF, Capacitor_Tantalum_SMD:CP_EIA-3528-21_Kemet-B, F.Cu at (103.4, 114.2)
- added C2: 330pF, Capacitor_SMD:C_0805_2012Metric_Pad1.18x1.45mm_HandSolder, F.Cu at (88.5, 97.0)
- added C3: 330pF, Capacitor_SMD:C_0805_2012Metric_Pad1.18x1.45mm_HandSolder, F.Cu at (88.5, 100.0)
- added C4: 330pF, Capacitor_SMD:C_0805_2012Metric_Pad1.18x1.45mm_HandSolder, F.Cu at (88.5, 103.0)
- added C5: 330pF, Capacitor_SMD:C_0805_2012Metric_Pad1.18x1.45mm_HandSolder, F.Cu at (88.5, 106.0)
- added D1: 19-213/Y2C-CQ2R2L/3T(CY), LED_SMD:LED_0603_1608Metric, F.Cu at (108.4, 113.3)
- added D2: CMOZ1L8, Diode_SMD:D_SOD-523, F.Cu at (92.7, 108.5)
- added D3: CMOZ1L8, Diode_SMD:D_SOD-523, F.Cu at (92.7, 111.0)
- added D4: 19-213/Y2C-CQ2R2L/3T(CY), LED_SMD:LED_0603_1608Metric, F.Cu at (108.4, 115.9)
- added D5: ESD5Z5V0, Diode_SMD:D_SOD-523, F.Cu at (92.7, 113.4)
- added F1: 500mA, Fuse:Fuse_1206_3216Metric, F.Cu at (97.9, 97.2)
- added F2: 500mA, Fuse:Fuse_1206_3216Metric, F.Cu at (97.9, 100.4)
- added F3: 1A5, Fuse:Fuse_1206_3216Metric, F.Cu at (97.9, 103.7)
- added FB1: GZ2012D601TF, Inductor_SMD:L_0805_2012Metric, F.Cu at (97.4, 115.7)
- added H1: MountingHole, MountingHole:MountingHole_3.2mm_M3_DIN965_Pad_TopBottom, F.Cu at (76.1, 66.1)
- added H2: MountingHole, MountingHole:MountingHole_3.2mm_M3_DIN965_Pad_TopBottom, F.Cu at (76.1, 73.2)
- added H3: MountingHole, MountingHole:MountingHole_3.2mm_M3_DIN965_Pad_TopBottom, F.Cu at (83.2, 66.1)
- added H4: MountingHole, MountingHole:MountingHole_3.2mm_M3_DIN965_Pad_TopBottom, F.Cu at (83.2, 73.2)
- added H5: MountingHole, MountingHole:MountingHole_3.2mm_M3_DIN965, F.Cu at (90.4, 66.1)
- added H6: MountingHole, MountingHole:MountingHole_3.2mm_M3_DIN965, F.Cu at (90.4, 73.2)
- added J2: 8918-P8B, usb3sun:Altronics_P1108_8918-P8B, F.Cu at (130.2, 111.1)
- added J3: USB-U267-BWS, Connector_USB:USB_A_CUI_UJ2-ADH-TH_Horizontal_Stacked, F.Cu at (86.6, 82.7)
- added Q1: 2N7002DW, Package_TO_SOT_SMD:SOT-363_SC-70-6, F.Cu at (93.0, 97.5)
- added Q3: 2N7002DW, Package_TO_SOT_SMD:SOT-363_SC-70-6, F.Cu at (93.0, 101.4)
- added Q4: MMBT2222A, Package_TO_SOT_SMD:SOT-23, F.Cu at (103.2, 97.9)
- added Q5: MMBT2222A, Package_TO_SOT_SMD:SOT-23, F.Cu at (103.2, 102.5)
- added Q7: 2N7002DW, Package_TO_SOT_SMD:SOT-363_SC-70-6, F.Cu at (93.0, 105.4)
- added R1: 20kΩ, Resistor_THT:R_Axial_DIN0207_L6.3mm_D2.5mm_P10.16mm_Horizontal, F.Cu at (39.4, 51.3)
- added R10: 22Ω, Resistor_THT:R_Axial_DIN0207_L6.3mm_D2.5mm_P10.16mm_Horizontal, F.Cu at (39.4, 87.7)
- added R11: 22Ω, Resistor_THT:R_Axial_DIN0207_L6.3mm_D2.5mm_P10.16mm_Horizontal, F.Cu at (39.4, 91.8)
- added R12: 22Ω, Resistor_THT:R_Axial_DIN0207_L6.3mm_D2.5mm_P10.16mm_Horizontal, F.Cu at (39.4, 95.8)
- added R13: 22Ω, Resistor_THT:R_Axial_DIN0207_L6.3mm_D2.5mm_P10.16mm_Horizontal, F.Cu at (39.4, 99.9)
- added R14: 6k2Ω, Resistor_THT:R_Axial_DIN0207_L6.3mm_D2.5mm_P10.16mm_Horizontal, F.Cu at (39.4, 103.9)
- added R15: 1kΩ, Resistor_THT:R_Axial_DIN0207_L6.3mm_D2.5mm_P10.16mm_Horizontal, F.Cu at (39.4, 108.0)
- added R16: 1kΩ, Resistor_THT:R_Axial_DIN0207_L6.3mm_D2.5mm_P10.16mm_Horizontal, F.Cu at (39.4, 112.0)
- added R17: 6k2Ω, Resistor_THT:R_Axial_DIN0207_L6.3mm_D2.5mm_P10.16mm_Horizontal, F.Cu at (39.4, 116.1)
- added R2: 20kΩ, Resistor_THT:R_Axial_DIN0207_L6.3mm_D2.5mm_P10.16mm_Horizontal, F.Cu at (39.4, 55.3)
- added R3: 20kΩ, Resistor_THT:R_Axial_DIN0207_L6.3mm_D2.5mm_P10.16mm_Horizontal, F.Cu at (39.4, 59.4)
- added R4: 20kΩ, Resistor_THT:R_Axial_DIN0207_L6.3mm_D2.5mm_P10.16mm_Horizontal, F.Cu at (39.4, 63.4)
- added R5: 20kΩ, Resistor_THT:R_Axial_DIN0207_L6.3mm_D2.5mm_P10.16mm_Horizontal, F.Cu at (39.4, 67.5)
- added R6: 20kΩ, Resistor_THT:R_Axial_DIN0207_L6.3mm_D2.5mm_P10.16mm_Horizontal, F.Cu at (39.4, 71.5)
- added R7: 20kΩ, Resistor_THT:R_Axial_DIN0207_L6.3mm_D2.5mm_P10.16mm_Horizontal, F.Cu at (39.4, 75.6)
- added R8: 20kΩ, Resistor_THT:R_Axial_DIN0207_L6.3mm_D2.5mm_P10.16mm_Horizontal, F.Cu at (39.4, 79.6)
- added R9: 20kΩ, Resistor_THT:R_Axial_DIN0207_L6.3mm_D2.5mm_P10.16mm_Horizontal, F.Cu at (39.4, 83.7)
- added SW1: TS-1187A-B-A-B, Button_Switch_SMD:SW_Push_1P1T_XKB_TS-1187A, F.Cu at (104.6, 108.7)
- added U1: Pico, CustomFootprints:Pico-BlackPill_Textless, F.Cu at (171.4, 110.5)
- added U2: SRV05-4, marbastlib-various:SOT-23-6-routable, F.Cu at (97.8, 107.6)
- added U3: SRV05-4, marbastlib-various:SOT-23-6-routable, F.Cu at (97.8, 112.1)
- added U4: MAX40200AUK, Package_TO_SOT_SMD:SOT-23-5, F.Cu at (108.2, 97.9)
- added U5: MAX40200AUK, Package_TO_SOT_SMD:SOT-23-5, F.Cu at (108.2, 102.5)
- added U6: ~, KiCad-SSD1306-0.91-OLED-4pin-128x32:SSD1306-0.91-OLED-4pin-128x32, F.Cu at (73.3, 50.0)
